File: tda8954-btl.sch (KiCad schematic (older format))
At the start: 89 parts, among them J1 Screw_Terminal_01x02, J10 Conn_01x01_Male, J2 Conn_01x01_Male, J3 Screw_Terminal_01x02, J4 Conn_01x01_Male, J5 Conn_01x01_Male, J6 Screw_Terminal_01x02, J7 Screw_Terminal_01x03, J8 Conn_01x01_Male, J9 Conn_01x01_Male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

Commit message: polishing; completed first pass layout
Parts:
- removed J3: Screw_Terminal_01x02, Terminals_Phoenix:TerminalBlock_Phoenix_MKDS1.5-2pol, symbol Connector:Screw_Terminal_01x02
- J10: footprint power:FASTON250P_5.08mm_male_vertical -> Mounting_Holes:MountingHole_3.2mm_M3_DIN965_Pad
Changed lines of the file:
@@
 	6300 2150 6300 2200
-$Comp
-L Connector:Screw_Terminal_01x02 J3
-U 1 1 61CAF432
-P 6500 2200
-F 0 "J3" H 6500 2300 50  0000 L CNN
-F 1 "Screw_Terminal_01x02" H 6400 2000 50  0001 L CNN
-F 2 "Terminals_Phoenix:TerminalBlock_Phoenix_MKDS1.5-2pol" H 6500 2200 50  0001 C CNN
-F 3 "~" H 6500 2200 50  0001 C CNN
-	1    6500 2200
-	1    0    0    -1
-$EndComp
 $Comp
 L Connector:Conn_01x01_Male J4
@@
 F 0 "J10" H 5558 3539 50  0000 C CNN
 F 1 "Conn_01x01_Male" H 5558 3540 50  0001 C CNN
-F 2 "power:FASTON250P_5.08mm_male_vertical" H 5450 3450 50  0001 C CNN
+F 2 "Mounting_Holes:MountingHole_3.2mm_M3_DIN965_Pad" H 5450 3450 50  0001 C CNN
 F 3 "~" H 5450 3450 50  0001 C CNN
 	1    5450 3450

Commit message: polishing, plotted gerbers
Parts:
- added R23, R24: 20, Resistors_SMD:R_0805, symbol Device:R
- J10: footprint Mounting_Holes:MountingHole_3.2mm_M3_DIN965_Pad -> power:FASTON250P_5.08mm_male_vertical
- R1, R6: value 10 -> 20
- R12, R18, R19: value 1k -> 3k9
Connections:
- net labels added: DIAG1
- net labels removed: TFB
- wire segments 251 -> 262
Changed lines of the file:
@@
 encoding utf-8
 Sheet 1 1
-Title ""
-Date ""
-Rev ""
-Comp ""
+Title "TDA8954 BTL appnote amplifier"
+Date "2021-11-28"
+Rev "A"
+Comp "Tyrrell Zaibatsu"
 Comment1 ""
 Comment2 ""
@@
 P 5050 1850
 F 0 "R1" V 4950 1850 50  0000 C CNN
-F 1 "10" V 5050 1850 50  0000 C CNN
+F 1 "20" V 5050 1850 50  0000 C CNN
 F 2 "Resistors_SMD:R_0805" V 4980 1850 50  0001 C CNN
 F 3 "~" H 5050 1850 50  0001 C CNN
@@
 $EndComp
 Wire Wire Line
-	5050 1700 5050 1500
+	5050 1700 5050 1650
 Connection ~ 5050 1500
 Text Label 4650 1500 2    50   ~ 0
@@
 P 5050 2650
 F 0 "R6" V 4950 2650 50  0000 C CNN
-F 1 "10" V 5050 2650 50  0000 C CNN
+F 1 "20" V 5050 2650 50  0000 C CNN
 F 2 "Resistors_SMD:R_0805" V 4980 2650 50  0001 C CNN
 F 3 "~" H 5050 2650 50  0001 C CNN
@@
 $EndComp
 Wire Wire Line
-	5050 2800 5050 3000
+	5050 2800 5050 2850
 Connection ~ 5050 3000
 $Comp
@@
 DIAG2
 Text Label 3350 1450 1    50   ~ 0
-TFB
+DIAG1
 Wire Wire Line
 	6050 2150 6300 2150
@@
 Connection ~ 5700 5050
 Text Label 5500 5050 0    50   ~ 0
-TFB
+DIAG1
 $Comp
 L Device:R R18
@@
 P 6400 5450
 F 0 "R18" V 6500 5450 50  0000 C CNN
-F 1 "1k" V 6400 5450 50  0000 C CNN
+F 1 "3k9" V 6400 5450 50  0000 C CNN
 F 2 "Resistors_SMD:R_0805" V 6330 5450 50  0001 C CNN
 F 3 "~" H 6400 5450 50  0001 C CNN
@@
 P 7650 5450
 F 0 "R19" V 7750 5450 50  0000 C CNN
-F 1 "1k" V 7650 5450 50  0000 C CNN
+F 1 "3k9" V 7650 5450 50  0000 C CNN
 F 2 "Resistors_SMD:R_0805" V 7580 5450 50  0001 C CNN
 F 3 "~" H 7650 5450 50  0001 C CNN
@@
 P 9150 4900
 F 0 "R12" V 9250 4900 50  0000 C CNN
-F 1 "1k" V 9150 4900 50  0000 C CNN
+F 1 "3k9" V 9150 4900 50  0000 C CNN
 F 2 "Resistors_SMD:R_0805" V 9080 4900 50  0001 C CNN
 F 3 "~" H 9150 4900 50  0001 C CNN
@@
 F 0 "J10" H 5558 3539 50  0000 C CNN
 F 1 "Conn_01x01_Male" H 5558 3540 50  0001 C CNN
-F 2 "Mounting_Holes:MountingHole_3.2mm_M3_DIN965_Pad" H 5450 3450 50  0001 C CNN
+F 2 "power:FASTON250P_5.08mm_male_vertical" H 5450 3450 50  0001 C CNN
 F 3 "~" H 5450 3450 50  0001 C CNN
 	1    5450 3450
@@
 Text Label 5700 3450 0    50   ~ 0
 HTSNK
+Wire Wire Line
+	3550 2950 3550 3250
+Text Label 3550 3200 1    50   ~ 0
+GND
+$Comp
+L Device:R R23
+U 1 1 62A9D397
+P 5150 1850
+F 0 "R23" V 5050 1850 50  0000 C CNN
+F 1 "20" V 5150 1850 50  0000 C CNN
+F 2 "Resistors_SMD:R_0805" V 5080 1850 50  0001 C CNN
+F 3 "~" H 5150 1850 50  0001 C CNN
+	1    5150 1850
+	-1   0    0    1
+$EndComp
+$Comp
+L Device:R R24
+U 1 1 62A9DAE4
+P 5150 2650
+F 0 "R24" V 5050 2650 50  0000 C CNN
+F 1 "20" V 5150 2650 50  0000 C CNN
+F 2 "Resistors_SMD:R_0805" V 5080 2650 50  0001 C CNN
+F 3 "~" H 5150 2650 50  0001 C CNN
+	1    5150 2650
+	-1   0    0    1
+$EndComp
+Wire Wire Line
+	5050 2450 5150 2450
+Wire Wire Line
+	5150 2450 5150 2500
+Wire Wire Line
+	5050 2850 5150 2850
+Wire Wire Line
+	5150 2850 5150 2800
+Connection ~ 5050 2850
+Wire Wire Line
+	5050 2850 5050 3000
+Wire Wire Line
+	5050 2050 5150 2050
+Wire Wire Line
+	5150 2050 5150 2000
+Wire Wire Line
+	5150 1700 5150 1650
+Wire Wire Line
+	5150 1650 5050 1650
+Connection ~ 5050 1650
+Wire Wire Line
+	5050 1650 5050 1500
 $EndSCHEMATC
